Commit message: greatly alleviate penetration

File: env/assets/box_lid.urdf (robot description, URDF)
Before this commit: robot box_lid.urdf, 2 links, 1 joints
Links:
- added link back; collision box size=0.01 0.18 0.03; visual box size=0.01 0.18 0.03
- added link front; collision box size=0.01 0.18 0.03; visual box size=0.01 0.18 0.03
- added link left; collision box size=0.23 0.01 0.03; visual box size=0.23 0.01 0.03
- added link right; collision box size=0.23 0.01 0.03; visual box size=0.23 0.01 0.03
- link lid: mass .1 -> .0212
- link top: geometry collision box size=0.23 0.18 0.01; visual box size=0.23 0.18 0.01
Joints:
- added joint back_joint: type fixed, parent top, child back, origin xyz=-0.11 0 -0.01 rpy=0 0 0
- added joint front_joint: type fixed, parent top, child front, origin xyz=0.11 0 -0.01 rpy=0 0 0
- added joint left_joint: type fixed, parent top, child left, origin xyz=0 -0.085 -0.01 rpy=0 0 0
- added joint right_joint: type fixed, parent top, child right, origin xyz=0 0.085 -0.01 rpy=0 0 0
- joint lid_joint: origin xyz=0 0 0.025 rpy=0 0 0 -> xyz=0 0 0.03 rpy=0 0 0
